File: MAM19.kicad_pcb (KiCad board)
At the start: 2 copper layers, 104 parts, among them J06 PWM/IR C, J101 GNDC1, J102 GNDC2, J103 GNDD1, J104 GNDD2, J105 PWM/IR D, J107 HOLD1, J108 HOLD2, J181 +18C, J182 +18D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

Commit message: ...
Parts:
- moved C904 19.2 mm to (119.5, 56.5)
- moved R701 11.2 mm to (73.5, 65.4)
- moved R702 11.2 mm to (70.9, 63.5)
- moved D703 0.80 mm to (91.6, 81.3)
Routing:
- net Net-(R406-Pad1): track 0.00 -> 2.68 mm
- net Net-(D403-Pad2): track 0.00 -> 1.78 mm
- net GND: track 415.7 -> 414.4 mm, vias 58 -> 36
- net (no net): vias 52 -> 0
