File: DRIVER_PANEL.kicad_pcb (KiCad board)
At the start: 2 copper layers, 261.3 x 104.4 mm, 132 parts, among them J103 GNDD1, J104 GNDD2, J105 PWM/IR D, J108 HOLD2, J182 +18D, J704 DRAINCH, J705 GATECH, J706 SOURCECH, U601 LM7815, U701 IR2127S, U702 UCC2732

Commit message: panels generated and pdfs exported
Parts:
- added C601: 1uF, Capacitor_Tantalum_SMD:CP_EIA-6032-20_AVX-F_Pad2.25x2.35mm_HandSolder, B.Cu at (181.9, 164.3)
- added C601: 1uF, Capacitor_Tantalum_SMD:CP_EIA-6032-20_AVX-F_Pad2.25x2.35mm_HandSolder, B.Cu at (54.9, 164.3)
- added C602: 100nF, Capacitor_SMD:C_0805_2012Metric_Pad1.15x1.40mm_HandSolder, B.Cu at (183.8, 167.5)
- added C602: 100nF, Capacitor_SMD:C_0805_2012Metric_Pad1.15x1.40mm_HandSolder, B.Cu at (56.8, 167.5)
- added C603: 100nF, Capacitor_SMD:C_0805_2012Metric_Pad1.15x1.40mm_HandSolder, B.Cu at (192.7, 152.9)
- added C603: 100nF, Capacitor_SMD:C_0805_2012Metric_Pad1.15x1.40mm_HandSolder, B.Cu at (65.7, 152.9)
- added C604: 1uF, Capacitor_Tantalum_SMD:CP_EIA-6032-20_AVX-F_Pad2.25x2.35mm_HandSolder, B.Cu at (192.7, 156.1)
- added C604: 1uF, Capacitor_Tantalum_SMD:CP_EIA-6032-20_AVX-F_Pad2.25x2.35mm_HandSolder, B.Cu at (65.7, 156.1)
- added C701: 100nF, Capacitor_SMD:C_0805_2012Metric_Pad1.15x1.40mm_HandSolder, B.Cu at (221.9, 156.7)
- added C701: 100nF, Capacitor_SMD:C_0805_2012Metric_Pad1.15x1.40mm_HandSolder, B.Cu at (94.9, 156.7)
- added C702: 100nF, Capacitor_SMD:C_0805_2012Metric_Pad1.15x1.40mm_HandSolder, F.Cu at (232.7, 149.7)
- added C702: 100nF, Capacitor_SMD:C_0805_2012Metric_Pad1.15x1.40mm_HandSolder, F.Cu at (105.7, 149.7)
- added C703: 100nF, Capacitor_SMD:C_0805_2012Metric_Pad1.15x1.40mm_HandSolder, F.Cu at (228.8, 161.2)
- added C703: 100nF, Capacitor_SMD:C_0805_2012Metric_Pad1.15x1.40mm_HandSolder, F.Cu at (101.8, 161.2)
- added C704: 100nF, Capacitor_SMD:C_0805_2012Metric_Pad1.15x1.40mm_HandSolder, F.Cu at (237.7, 152.9)
- added C704: 100nF, Capacitor_SMD:C_0805_2012Metric_Pad1.15x1.40mm_HandSolder, F.Cu at (110.7, 152.9)
- added C705: 1uF, Capacitor_SMD:C_0805_2012Metric_Pad1.15x1.40mm_HandSolder, F.Cu at (241.6, 152.9)
- added C705: 1uF, Capacitor_SMD:C_0805_2012Metric_Pad1.15x1.40mm_HandSolder, F.Cu at (114.6, 152.9)
- added C706: 10uF, Capacitor_Tantalum_SMD:CP_EIA-6032-20_AVX-F_Pad2.25x2.35mm_HandSolder, B.Cu at (239.6, 153.5)
- added C706: 10uF, Capacitor_Tantalum_SMD:CP_EIA-6032-20_AVX-F_Pad2.25x2.35mm_HandSolder, B.Cu at (112.6, 153.5)
- added D601: LL4148, Diode_SMD:D_MiniMELF_Handsoldering, B.Cu at (186.9, 170.1)
- added D601: LL4148, Diode_SMD:D_MiniMELF_Handsoldering, B.Cu at (59.9, 170.1)
- added D701: BAV102, Diode_SMD:D_MiniMELF_Handsoldering, F.Cu at (225.7, 147.2)
- added D701: BAV102, Diode_SMD:D_MiniMELF_Handsoldering, F.Cu at (98.7, 147.2)
- added D702: BYD77, Diode_SMD:D_MELF, B.Cu at (220.0, 151.6)
- added D702: BYD77, Diode_SMD:D_MELF, B.Cu at (93.0, 151.6)
- added D703: ES3B, Diode_SMD:D_SMC_Handsoldering, F.Cu at (244.7, 145.9)
- added D703: ES3B, Diode_SMD:D_SMC_Handsoldering, F.Cu at (117.7, 145.9)
- added DZ701: 15V, Diode_SMD:D_MiniMELF_Handsoldering, F.Cu at (249.2, 159.3)
- added DZ701: 15V, Diode_SMD:D_MiniMELF_Handsoldering, F.Cu at (122.2, 159.3)
- added J103: GNDD1, Connector_PinHeader_2.54mm:PinHeader_2x02_P2.54mm_Vertical, F.Cu at (197.1, 176.7)
- added J103: GNDD1, Connector_PinHeader_2.54mm:PinHeader_2x02_P2.54mm_Vertical, F.Cu at (70.1, 176.7)
- added J104: GNDD2, Connector_PinHeader_2.54mm:PinHeader_2x02_P2.54mm_Vertical, B.Cu at (191.7, 140.8)
- added J104: GNDD2, Connector_PinHeader_2.54mm:PinHeader_2x02_P2.54mm_Vertical, B.Cu at (64.7, 140.8)
- added J105: PWM/IR D, Connector_PinSocket_2.54mm:PinSocket_1x04_P2.54mm_Vertical_SMD_Pin1Left, F.Cu at (230.1, 167.5)
- added J105: PWM/IR D, Connector_PinSocket_2.54mm:PinSocket_1x04_P2.54mm_Vertical_SMD_Pin1Left, F.Cu at (103.1, 167.5)
- added J108: HOLD2, Connector_PinHeader_2.54mm:PinHeader_2x02_P2.54mm_Vertical, B.Cu at (171.7, 182.4)
- added J108: HOLD2, Connector_PinHeader_2.54mm:PinHeader_2x02_P2.54mm_Vertical, B.Cu at (44.7, 182.4)
- added J182: +18D, Connector_PinHeader_2.54mm:PinHeader_2x02_P2.54mm_Vertical, F.Cu at (188.8, 176.7)
- added J182: +18D, Connector_PinHeader_2.54mm:PinHeader_2x02_P2.54mm_Vertical, F.Cu at (61.8, 176.7)
- added J704: DRAINCH, Connector_PinHeader_2.54mm:PinHeader_2x02_P2.54mm_Vertical, B.Cu at (171.7, 140.2)
- added J704: DRAINCH, Connector_PinHeader_2.54mm:PinHeader_2x02_P2.54mm_Vertical, B.Cu at (44.7, 140.2)
- added J705: GATECH, Connector_PinHeader_2.54mm:PinHeader_2x02_P2.54mm_Vertical, B.Cu at (247.5, 140.7)
- added J705: GATECH, Connector_PinHeader_2.54mm:PinHeader_2x02_P2.54mm_Vertical, B.Cu at (120.5, 140.7)
- added J706: SOURCECH, Connector_PinHeader_2.54mm:PinHeader_2x02_P2.54mm_Vertical_SMD, B.Cu at (248.5, 176.4)
- added J706: SOURCECH, Connector_PinHeader_2.54mm:PinHeader_2x02_P2.54mm_Vertical_SMD, B.Cu at (121.5, 176.4)
- added R701: 22K, Resistor_SMD:R_0805_2012Metric_Pad1.15x1.40mm_HandSolder, F.Cu at (228.9, 149.7)
- added R701: 22K, Resistor_SMD:R_0805_2012Metric_Pad1.15x1.40mm_HandSolder, F.Cu at (101.9, 149.7)
- added R702: 10K, Resistor_SMD:R_0805_2012Metric_Pad1.15x1.40mm_HandSolder, F.Cu at (226.9, 152.3)
- added R702: 10K, Resistor_SMD:R_0805_2012Metric_Pad1.15x1.40mm_HandSolder, F.Cu at (99.9, 152.3)
- added R703: 820, Resistor_SMD:R_0805_2012Metric_Pad1.15x1.40mm_HandSolder, F.Cu at (228.9, 163.1)
- added R703: 820, Resistor_SMD:R_0805_2012Metric_Pad1.15x1.40mm_HandSolder, F.Cu at (101.9, 163.1)
- added R704: 0, Resistor_SMD:R_0805_2012Metric_Pad1.15x1.40mm_HandSolder, F.Cu at (233.9, 154.8)
- added R704: 0, Resistor_SMD:R_0805_2012Metric_Pad1.15x1.40mm_HandSolder, F.Cu at (106.9, 154.8)
- added R705: 4R7, Resistor_SMD:R_0805_2012Metric_Pad1.15x1.40mm_HandSolder, F.Cu at (244.7, 152.3)
- added R705: 4R7, Resistor_SMD:R_0805_2012Metric_Pad1.15x1.40mm_HandSolder, F.Cu at (117.7, 152.3)
- added R706: 10, Resistor_SMD:R_0805_2012Metric_Pad1.15x1.40mm_HandSolder, F.Cu at (246.0, 156.1)
- added R706: 10, Resistor_SMD:R_0805_2012Metric_Pad1.15x1.40mm_HandSolder, F.Cu at (119.0, 156.1)
- added R707: 10K, Resistor_SMD:R_0805_2012Metric_Pad1.15x1.40mm_HandSolder, F.Cu at (251.1, 159.3)
- added R707: 10K, Resistor_SMD:R_0805_2012Metric_Pad1.15x1.40mm_HandSolder, F.Cu at (124.1, 159.3)
- added U601: LM7815, KicadZeniteSolarLibrary18:TO-220-3_Horizontal_TabDown_SMD, B.Cu at (191.4, 165.6)
- added U601: LM7815, KicadZeniteSolarLibrary18:TO-220-3_Horizontal_TabDown_SMD, B.Cu at (64.4, 165.6)
- added U701: IR2127S, Package_SO:SOIC-8_3.9x4.9mm_P1.27mm, F.Cu at (228.9, 156.7)
- added U701: IR2127S, Package_SO:SOIC-8_3.9x4.9mm_P1.27mm, F.Cu at (101.9, 156.7)
- added U702: UCC2732, Package_SO:MSOP-8-1EP_3x3mm_P0.65mm_EP2.54x2.8mm_ThermalVias, F.Cu at (240.9, 156.1)
- added U702: UCC2732, Package_SO:MSOP-8-1EP_3x3mm_P0.65mm_EP2.54x2.8mm_ThermalVias, F.Cu at (113.9, 156.1)
- moved D702 14.2 mm to (250.6, 80.5)
- moved R702 14.2 mm to (250.0, 87.5)
- moved R705 14.2 mm to (250.0, 105.3)
- moved C602 14.2 mm to (234.8, 44.3)
- moved C604 14.2 mm to (246.2, 53.2)
- moved J105 14.2 mm to (234.8, 90.7)
- moved J704 14.2 mm to (262.1, 32.2)
- moved R706 14.2 mm to (246.2, 106.6)
- moved U702 14.2 mm to (246.2, 101.5)
- moved C702 14.2 mm to (252.5, 93.2)
- moved C703 14.2 mm to (241.1, 89.4)
- moved D701 14.2 mm to (255.1, 86.2)
- moved J182 14.2 mm to (225.6, 49.4)
- moved J706 14.2 mm to (225.9, 109.1)
- moved R701 14.2 mm to (252.5, 89.4)
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Routing:
- net (no net): track 0.00 -> 1046.6 mm, vias 16 -> 94
- added copper zone on B.Cu, net (none)
- added copper zone on F.Cu, net (none)
Other:
- board size 261.3 x 104.4 mm -> 238.4 x 171.7 mm
